File: asic-3up-0.kicad_sch (KiCad schematic)
At the start: 64 parts, among them J18 Conn_01x01, J3 Conn_01x01, J4 Conn_01x01, U28 MCP1824T-1202E/OT, U29 MCP1824T-1202E/OT, U30 MCP1824T-1202E/OT, U32 MCP1824T-0802E, U42 MCP1824T-0802E, U43 MCP1824T-0802E, U45 BM1362AC_MODE1, U46 BM1362AC_MODE0, U47 BM1362AC_MODE1

Commit message: manually imported BOM changes from PR #42. generated manufacturing files.
Parts:
- R64: PARTNO RC0402FR-072KL -> RC0402FR-071KL
Changed lines of the file:
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@@
 			)
 		)
-		(property "PARTNO" "RC0402FR-072KL"
+		(property "PARTNO" "RC0402FR-071KL"
 			(at 195.58 66.04 0)
 			(effects
